File: Meter_PCB_V1.brd (EAGLE design)
At the start: 43 x 51.1 mm, 63 parts, among them CN1 MicroB USB, IC1 ATMEGA32U4-MU, IC2 LMV358MM, IC4 LIS3DH, U1 SPW2430, U2 MBT40, U4 MCP73831T-2ACI/OT, U5 SPX3819-3.3, X1 JSTPH, Y1 8MHz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

Commit message: finished board design
Parts:
- removed C12, C13, C15: 10µF, microbuilder:0805-NO
- removed C14, C16: 1uF, microbuilder:0603-NO
- removed CHG: ORANGE, microbuilder:CHIPLED_0805_NOOUTLINE
- removed D5: MBR120, microbuilder:SOD-123
- removed R19: 1K, microbuilder:0603-NO
- removed R20: 10K\, microbuilder:0603-NO
- removed R21, R23, R24: 100K, microbuilder:0603-NO
- removed TP6, TP7, TP8: MISO, microbuilder:TESTPOINT_ROUND_1.5MM
- removed U4: MCP73831T-2ACI/OT, microbuilder:SOT23-5
- removed U5: SPX3819-3.3, microbuilder:SOT23-5
- removed X1: JSTPH, microbuilder:JSTPH2
- moved C11 52.2 mm to (7.81, -15.8), turned to 270 degrees
- moved C10 51.5 mm to (-3.19, -18.2), turned to 180 degrees
- moved R7 51.3 mm to (-7.19, -18.3), turned to 180 degrees
- moved D3 51.3 mm to (-11.0, -18.0), turned to 90 degrees
- moved Y2 46.4 mm to (-1.48, -14.4), turned to 180 degrees
- moved DFU 45.7 mm to (8.25, -10.5), turned to 90 degrees
- moved U2 41.4 mm to (-3.74, -11.1), turned to 90 degrees
- moved R17 34.5 mm to (4.00, -4.00), turned to 0 degrees
- moved R16 32.6 mm to (0.00, -4.00), turned to 180 degrees
- moved D4 32.1 mm to (-11.0, -4.35), turned to 90 degrees
- moved R12 31.3 mm to (-7.19, -4.11), turned to 180 degrees
- moved TP5 12.0 mm to (-8.00, 14.0), flipped to the bottom
- moved R14 11.4 mm to (7.08, -4.81)
- moved TP9 11.4 mm to (-8.00, 16.0), flipped to the bottom
- moved J-L 10.0 mm to (-13.0, 15.0)
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Connections:
- removed net +3V3: C14.1, C15.1, U5.5
- removed net 9: R21.2, R23.1
- removed net EN: R24.2, U5.3
- removed net N$16: CHG.C, R19.1
- removed net N$17: R19.2, U4.1
- removed net N$18: R20.1, U4.5
- net AREF: no longer C16.1
- net FCTRYRST_3V: no longer TP8.P$1
- net GND: no longer C12.2, C13.2, C14.2, C15.2, C16.2, R20.2, R23.2, U4.2, U5.2, X1.1
- net SWCLK: no longer TP6.P$1
- net SWDIO/RST_3V: no longer TP7.P$1
- net VBAT: no longer C12.1, D5.A, R21.1, U4.3, X1.2
- net VBUS: no longer C13.1, CHG.A, D5.C, R24.1, U4.4, U5.1
Routing:
- net SWCLK: track 9.33 -> 4.13 mm
- net SWDIO/RST_3V: track 8.77 -> 3.81 mm
- net MISO: track 29.4 -> 26.4 mm
- net FCTRYRST_3V: track 9.18 -> 6.59 mm
- net D8: track 15.9 -> 16.7 mm
- net A4_SOUND_SENSE: track 31.6 -> 32.3 mm
Other:
- board size 43 x 51.1 mm -> 31.1 x 46.1 mm
