File: Meter_PCB_V1.sch (EAGLE design)
At the start: 62 parts, among them CN1 MicroB USB, IC1 ATMEGA32U4-MU, IC2 LMV358MM, IC4 LIS3DH, U1 SPW2430, U2 MBT40, U4 MCP73831T-2ACI/OT, U5 SPX3819-3.3, X1 JSTPH, Y1 8MHz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

Commit message: finished board design
Parts:
- removed C12, C13, C15: 10µF, microbuilder:CAP_CERAMIC0805-NOOUTLINE
- removed C14, C16: 1uF, microbuilder:CAP_CERAMIC0603_NO
- removed CHG: ORANGE, microbuilder:LED0805_NOOUTLINE
- removed D5: MBR120, microbuilder:DIODE-SCHOTTKYSOD-123
- removed R19: 1K, microbuilder:RESISTOR_0603_NOOUT
- removed R20: 10K\, microbuilder:RESISTOR_0603_NOOUT
- removed R21, R23, R24: 100K, microbuilder:RESISTOR_0603_NOOUT
- removed TP6, TP7, TP8: MISO, microbuilder:TESTPOINTROUND1.5MM
- removed U4: MCP73831T-2ACI/OT, microbuilder:MCP73831/2
- removed U5: SPX3819-3.3, microbuilder:VREG_SOT23-5
- removed X1: JSTPH, microbuilder:CON_JST_PH_2PIN
Connections:
- removed net +3V3: C14.1, C15.1, U5.OUT
- removed net 9: R21.2, R23.1
- removed net EN: R24.2, U5.EN
- removed net N$16: CHG.C, R19.1
- removed net N$17: R19.2, U4.STAT
- removed net N$18: R20.1, U4.PROG
- net AREF: no longer C16.1
- net FCTRYRST_3V: no longer TP8.P$1
- net GND: no longer C12.2, C13.2, C14.2, C15.2, C16.2, R20.2, R23.2, U4.VSS, U5.GND, X1.1
- net SWCLK: no longer TP6.P$1
- net SWDIO/RST_3V: no longer TP7.P$1
- net VBAT: no longer C12.1, D5.A, R21.1, U4.VBAT, X1.2
- net VBUS: no longer C13.1, CHG.A, D5.C, R24.1, U4.VDD, U5.IN
Other:
- note removed: "1.0K = 1000mA"
- note removed: "10K = 100mA"
- note removed: "2.0K = 500mA"
- note removed: "5.0K = 200mA"
- note removed: "LIPO & CHARGING"
- note removed: "POWER AND FILTERING"
