File: Meter_PCB_V2.sch (EAGLE design)
At the start: 60 parts, among them CN1 MicroB USB, IC1 ATMEGA32U4-MU, IC2 LMV358MM, IC4 LIS3DH, U1 SPW2430, U2 MBT40, U4 MCP73831T-2ACI/OT, U5 SPX3819-3.3, X1 JSTPH, Y1 8MHz, Y2 32.768kHz (535-9166-2-ND)

Commit message: finished board design
Parts:
- removed C12, C13, C15: 10µF, microbuilder:CAP_CERAMIC0805-NOOUTLINE
- removed C14, C16: 1uF, microbuilder:CAP_CERAMIC0603_NO
- removed CHG: ORANGE, microbuilder:LED0805_NOOUTLINE
- removed D5: MBR120, microbuilder:DIODE-SCHOTTKYSOD-123
- removed DFU: KMR2, microbuilder:SWITCH_TACT_SMT4.6X2.8
- removed J-L, J-R: (no value), SparkFun-Connectors:CONN_04
- removed R14: 2K, microbuilder:RESISTOR0805_NOOUTLINE
- removed R19: 1K, microbuilder:RESISTOR_0603_NOOUT
- removed R20: 10K\, microbuilder:RESISTOR_0603_NOOUT
- removed R21, R23, R24: 100K, microbuilder:RESISTOR_0603_NOOUT
- removed U4: MCP73831T-2ACI/OT, microbuilder:MCP73831/2
- removed U5: SPX3819-3.3, microbuilder:VREG_SOT23-5
- removed X1: JSTPH, microbuilder:CON_JST_PH_2PIN
- added BATT: 3-6VDC, microbuilder:CON_JST_PH_2PIN
- added C2, C3, C5, C6, C7: 1uF, microbuilder:CAP_CERAMIC0603_NO
- added C4, C8: 10uF, microbuilder:CAP_CERAMIC0805-NOOUTLINE
- added D1, D2: SCHOTTKY (1A), microbuilder:DIODESOD-123
- added NEOPIXEL-L, NEOPIXEL-R: (no value), SparkFun-Connectors:CONN_04
- added R18: 0, microbuilder:RESISTOR_0603_NOOUT
- added RESET1: KMR2, microbuilder:SWITCH_TACT_SMT4.6X2.8
- added SW2: EVQQ, microbuilder:SWITCH_TACT_SMT_EVQQ2_SMALL
- added TP5: SWCLK, microbuilder:TESTPOINTROUND1.5MM
- added TP9: SDA, microbuilder:TESTPOINTROUND1.5MM
- added U3: AP2112K-3.3, microbuilder:VREG_SOT23-5
- R13: device microbuilder:RESISTOR0805_NOOUTLINE -> microbuilder:RESISTOR_0603_NOOUT
- R16: value 0 -> 2K; device microbuilder:RESISTOR_0603_NOOUT -> microbuilder:RESISTOR0805_NOOUTLINE
- R4: value 1M -> 10K; device microbuilder:RESISTOR_4PACK_NO -> microbuilder:RESISTOR0805_NOOUTLINE
- TP6: value MISO -> SWDIO
- TP7: value MISO -> FACTORYRST
- TP8: value MISO -> SCL
Connections:
- removed net +3V3: C14.1, C15.1, U5.OUT
- removed net 9: R21.2, R23.1
- removed net A0_TEMP_SENSE: IC1.PF7(ADC7(TDI)
- removed net A2: IC1.PF5(ADC5/TMS)
- removed net A3_SWITCH: IC1.PF4(ADC4/TCK)
- removed net A5_LIGHT_SENSE: IC1.PF0(ADC0)
- removed net EN: R24.2, U5.EN
- removed net LEFTBUTTON: IC1.PD4(ICP1/ADC8)
- removed net N$16: CHG.C, R19.1
- removed net N$17: R19.2, U4.STAT
- removed net N$18: R20.1, U4.PROG
- removed net NEOPIX: IC1.PB0(SS)
- removed net SPEAKER: IC1.PC6(OC3A/!OC4A)
- removed net VBAT: C12.1, CN1.VBUS, D5.A, J-L.3, J-R.2, R21.1, U4.VBAT, X1.2
- removed net VBUS: C13.1, CHG.A, D5.C, IC1.VBUS, R24.1, U4.VDD, U5.IN
- new net +5V: CN1.VBUS, D1.A, IC1.VBUS
- new net N$7: BATT.2, D2.A
- new net VCC: C4.1, C5.1, D1.C, D2.C, NEOPIXEL-L.2, NEOPIXEL-R.3, U3.EN, U3.IN
- net 3.3V: now also C2.1, C3.1, C6.1, C7.1, C8.1, NEOPIXEL-L.1, R4.1, SW2.S, SW2.S1, U3.OUT; no longer J-L.4, J-R.1, R13.1
- net A1_RIGHTBUTTON: now also R13.2, SW2.P, SW2.P1
- net AREF: no longer C16.1
- net D0/RX: now also R18.2; no longer R17.2
- net D1/TX: now also R17.2; no longer R16.2
- net D10: now also R22G$4.2
- net D12: now also R16.2, R22G$3.2; no longer R14.2, R4G$2.2
- net D2_SDA: now also R15G$2.2, TP9.P$1
- net D3_SCL: now also R15G$1.2, TP8.P$1
- net D6: now also NEOPIXEL-L.3; no longer J-R.3
- net D9: now also NEOPIXEL-R.2; no longer J-L.2
- net DFU: now also R4.2, RESET1.S, RESET1.S1; no longer DFU.P, DFU.P1, R13.2
- net FCTRYRST_3V: now also TP7.P$1; no longer TP8.P$1
- net GND: now also BATT.1, C2.2, C3.2, C4.2, C5.2, C6.2, C7.2, C8.2, NEOPIXEL-L.4, NEOPIXEL-R.1, R13.1, RESET1.P, RESET1.P1, U3.GND; no longer C12.2, C13.2, C14.2, C15.2, C16.2, DFU.S, DFU.S1, J-L.1, J-R.4, R20.2, R23.2, U4.VSS, U5.GND, X1.1
- net MODE: now also R16.1; no longer R14.1
- net RXI: now also R17.1; no longer R16.1
- net SWCLK: now also TP5.P$1; no longer TP6.P$1
- net SWDIO/RST_3V: now also TP6.P$1; no longer TP7.P$1
- net TXLED: now also R15G$1.1, R15G$2.1, R22G$3.1, R22G$4.1; no longer R4G$2.1
- net TXO: now also R18.1; no longer R17.1
Other:
- note added: "3.3V Reg"
- note added: "ATMEGA32u4 MICROCONTROLLER"
- note added: "JST Battery In"
- note added: "LEDs"
- note added: "Tact Switch"
- note removed: "1.0K = 1000mA"
- note removed: "10K = 100mA"
- note removed: "2.0K = 500mA"
- note removed: "5.0K = 200mA"
- note removed: "LIPO & CHARGING"
- note removed: "MICROCONTROLLER"
- note removed: "POWER AND FILTERING"
- moved on the sheet: C1, C10, C11, C9, CN1, D3, D4, IC1, IC2A, IC2B, IC4, L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
